File: digilab.kicad_sch (KiCad schematic)
At the start: 86 parts, among them J1 AE, J2 OUT, J3 IN, Q1 BC636, Q10 BC636, Q2 BC636, Q3 BC636, Q4 BC636, Q5 BC636, Q6 BC636, Q7 BC636, Q8 BC636, Q9 BC636, U1 PC817, U10 PC817, U11 PC817, U12 PC817, U13 PC817, U14 PC817, U15 PC817, U16 PC817, U17 PC817, U18 PC817, U19 PC817, U2 PC817, U20 PC817, U3 PC817, U4 PC817, U5 PC817, U6 PC817, U7 PC817, U8 PC817, U9 PC817

Commit message: DigiLab V1.0
Other:
- note added: "This source describes Open Hardware and is licensed under the CERN-OHL-S v2. You may redistribute and modify this file under the terms of the CERN-OHL-S v2. A copy of the license is available at https://ohwr.org/cernohl"
Changed lines of the file:
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@@
+		)
+	)
+	(text "This source describes Open Hardware and is licensed under the CERN-OHL-S v2.\nYou may redistribute and modify this file under the terms of the CERN-OHL-S v2.\nA copy of the license is available at https://ohwr.org/cernohl"
+		(exclude_from_sim no)
+		(at 231.14 174.244 0)
+		(effects
+			(font
+				(size 1.524 1.524)
+			)
 		)
 	)
